File: pebble/pebble.kicad_pcb (KiCad board)
At the start: 4 copper layers, 129 x 129 mm, 160 parts, among them J1 UART, J2 GPS, J3 USB_C_Receptacle_USB2.0_16P, J4 BAT, J5 Conn_01x03_Pin, Q1 BSS84, Q2 BSS123, U1 TPS61023DRLR, U2 TPS563200, U3 ESP32-C6-MINI-1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

Commit message: finalize rev0
Parts:
- added J6: ON, Connector_PinHeader_1.27mm:PinHeader_1x02_P1.27mm_Vertical, F.Cu at (142.5, 70.8)
- added J7: ON, Connector_PinHeader_1.27mm:PinHeader_1x02_P1.27mm_Vertical, F.Cu at (143.8, 67.7)
- added SW1: SW_Reed, kicad-symbols:59170-1-S-00-D, B.Cu at (135.9, 85.9)
- moved J4 3.42 mm to (143.7, 75.1), turned to 180 degrees
Connections:
- C26 pad 1: Net-(J4-Pin_2) -> Net-(J6-Pin_2)
- J3 pad A6: /charger/DN_in -> /charger/DP_in
- J3 pad A7: /charger/DP_in -> /charger/DN_in
- J3 pad B6: /charger/DN_in -> /charger/DP_in
- J3 pad B7: /charger/DP_in -> /charger/DN_in
- R18 pad 2: Net-(J4-Pin_2) -> Net-(J6-Pin_2)
- U7 pad 13: Net-(J4-Pin_2) -> Net-(J6-Pin_2)
- U7 pad 14: Net-(J4-Pin_2) -> Net-(J6-Pin_2)
Routing:
- net Net-(J6-Pin_2): track 0.00 -> 36.2 mm, vias 0 -> 37
- net Net-(J4-Pin_2): track 1.56 -> 30.3 mm, vias 36 -> 0
- net Net-(JP2-B): track 63.6 -> 62.2 mm
- added copper zone on B.Cu, net Net-(J6-Pin_2)
- added copper zone on F.Cu, net Net-(J6-Pin_2)
- removed copper zone on B.Cu, net Net-(J4-Pin_2)
- removed copper zone on F.Cu, net Net-(J4-Pin_2)
Other:
- board text added: "BATTERY"
- board text added: "ON"
- board text added: "Pebble rev0 designed by @Yatekii"

Commit message: put charger leds on the back layer, position imu precisely, simplify schema, tapeout
Parts:
- added H1: MountingHole, MountingHole:MountingHole_3.2mm_M3, F.Cu at (118.2, 68.2)
- added H2: MountingHole, MountingHole:MountingHole_3.2mm_M3, F.Cu at (181.8, 68.2)
- added H3: MountingHole, MountingHole:MountingHole_3.2mm_M3, F.Cu at (181.8, 131.8)
- added H4: MountingHole, MountingHole:MountingHole_3.2mm_M3, F.Cu at (118.2, 131.8)
- D73, D74, R14, R15: moved to B.Cu
- moved D74 36.2 mm to (143.0, 102.4), turned to 0 degrees
- moved D73 34.5 mm to (143.0, 100.8), turned to 0 degrees
- moved R15 31.8 mm to (140.4, 102.4), turned to 180 degrees
- moved R14 30.1 mm to (140.4, 100.8), turned to 180 degrees
- moved C19 17.9 mm to (194.7, 102.5), turned to 180 degrees
- moved C14 17.1 mm to (188.5, 100.1)
- moved C12 17.0 mm to (191.5, 100.1)
- moved U6 17.0 mm to (190.0, 100.0)
- moved C17 16.8 mm to (190.0, 101.5)
- moved C20 16.8 mm to (192.8, 100.0)
- moved U4 16.7 mm to (195.0, 100.0)
- moved R29 13.3 mm to (197.7, 100.5), turned to 180 degrees
- moved R28 12.2 mm to (197.7, 99.5)
- moved R25 8.13 mm to (121.2, 73.5), turned to 0 degrees
- moved C24 7.37 mm to (147.9, 83.3)
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Routing:
- net VBUS: track 39.4 -> 3.06 mm
- net /charger/CHRG: track 47.1 -> 18.1 mm, vias 2 -> 1
- net /charger/INOK: track 47.4 -> 20.2 mm, vias 2 -> 1
- net +5V: track 20.2 -> 2.10 mm
- net +3V3: track 153.3 -> 138.6 mm, vias 142 -> 139
- net Net-(U2-SW): track 18.5 -> 5.69 mm
- net /IMU_INT1: track 34.3 -> 21.7 mm, vias 0 -> 2
- net /IMU_INT2: track 31.8 -> 24.0 mm, vias 0 -> 2
- net Net-(U7-PVL): track 8.92 -> 1.45 mm
- net Net-(C25-Pad2): track 5.99 -> 0.00 mm
- net /MAG_INT: track 26.9 -> 21.3 mm, vias 0 -> 2
- net /SDA2: track 39.1 -> 33.8 mm
- net /BMM_SDA: track 12.1 -> 6.96 mm
- net /BMM_SCL: track 10.7 -> 5.71 mm
- net GND: track 48.5 -> 51.8 mm, vias 104 -> 106
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- added copper zone on B.Cu, net Net-(C25-Pad2)
- removed copper zone on In1.Cu, net +BATT
