File: pebble/pebble.kicad_sch (KiCad schematic)
At the start: 126 parts, among them J1 UART, J2 GPS, J5 Conn_01x03_Pin, Q1 BSS84, Q2 BSS123, U1 TPS61023DRLR, U2 TPS563200, U3 ESP32-C6-MINI-1, U4 BMI270, U5 MAX-M8Q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

Commit message: put charger leds on the back layer, position imu precisely, simplify schema, tapeout
Parts:
- added H1, H2, H3, H4: MountingHole, MountingHole:MountingHole_3.2mm_M3, symbol Mechanical:MountingHole
- C18: value C_Small -> 1n
- L3: value TBD -> 27n; Part (none) -> LQG15HS27NJ02
