File: pebble/usb-fast-charger.kicad_sch (KiCad schematic)
At the start: 35 parts, among them J3 USB_C_Receptacle_USB2.0_16P, J4 BAT, U7 MAX77751CEFG+, U8 LPV521, U9 MAX4906ELB+T

Commit message: finalize rev0
Parts:
- added J6, J7: ON, Connector_PinHeader_1.27mm:PinHeader_1x02_P1.27mm_Vertical, symbol Connector:Conn_01x02_Pin
- added SW1: SW_Reed, kicad-symbols:59170-1-S-00-D, symbol Switch:SW_Reed
Connections:
- net DN_in: now also J3.A7 (D-), J3.B7 (D-); no longer J3.A6 (D+), J3.B6 (D+)
- net DP_in: now also J3.A6 (D+), J3.B6 (D+); no longer J3.A7 (D-), J3.B7 (D-)
- net at C26.1, R18.2, U7.13 (BATT)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: now also J6.2 (Pin_2), J7.1 (Pin_1), SW1.1; no longer J4.2 (Pin_2)
- new net: J4.2 (Pin_2), J6.1 (Pin_1), J7.2 (Pin_2), SW1.2
Other:
- moved on the sheet: BT1, J4
