File: hardware/pebble.kicad_pcb (KiCad board)
At the start: 4 copper layers, 129 x 129 mm, 167 parts, among them J1 UART, J2 GPS, J3 USB_C_Receptacle_USB2.0_16P, J4 BAT, J5 Conn_01x03_Pin, J6 ON, J7 ON, Q1 BSS84, Q2 BSS123, SW1 SW_Reed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

Commit message: add nix flake and initial esp32-c6 project structure with probe-rs and defmt
Parts:
- C18: value C_Small -> 1n
- C24: value 2.2u -> 2.2uF
- C25: value 100n -> 100nF
- C27, C28, C29: value 10u -> 10uF
- C31: value 22u -> 22uF
- L3: value TBD -> 27n
- L4: value 0.47u -> 0.47uH
Changed lines of the file:
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@@
 			)
 		)
+		(property "LCSC" "C2908590"
+			(at 0 0 90)
+			(unlocked yes)
+			(layer "F.Fab")
+			(hide yes)
+			(effects
+				(font
+					(size 1 1)
+					(thickness 0.15)
+				)
+			)
+		)
 		(property ki_fp_filters "21-100385_90-100128_MXM")
 		(sheetname "/charger/")
@@
 			)
 		)
+		(property "LCSC Part #" "C17225907"
+			(at 0 0 0)
+			(unlocked yes)
+			(layer "F.Fab")
+			(hide yes)
+			(effects
+				(font
+					(size 1 1)
+					(thickness 0.15)
+				)
+			)
+		)
 		(property ki_fp_filters "BGA9_BMM350_BOS BGA9_BMM350_BOS-M BGA9_BMM350_BOS-L")
 		(sheetname "/")
@@
 			)
 		)
+		(property "LCSC Part #" "C97253"
+			(at 0 0 180)
+			(unlocked yes)
+			(layer "F.Fab")
+			(hide yes)
+			(effects
+				(font
+					(size 1 1)
+					(thickness 0.15)
+				)
+			)
+		)
 		(property ki_fp_filters "ESP32?C6?MINI?1*")
 		(sheetname "/")
@@
 			)
 		)
+		(property "LCSC Part #" "C919459"
+			(at 0 0 270)
+			(unlocked yes)
+			(layer "F.Fab")
+			(hide yes)
+			(effects
+				(font
+					(size 1 1)
+					(thickness 0.15)
+				)
+			)
+		)
 		(property ki_fp_filters "DRL0006A")
 		(sheetname "/")
@@
 			)
 		)
-		(property "Value" "0.47u"
+		(property "Value" "0.47uH"
 			(at 0 0 90)
 			(unlocked yes)
@@
 			)
 		)
-		(property "Value" "100n"
+		(property "Value" "100nF"
 			(at 0 1.16 0)
 			(layer "F.Fab")
@@
 			)
 		)
+		(property "LCSC Part #" "C2836813"
+			(at 0 0 270)
+			(unlocked yes)
+			(layer "F.Fab")
+			(hide yes)
+			(effects
+				(font
+					(size 1 1)
+					(thickness 0.15)
+				)
+			)
+		)
 		(property ki_fp_filters "BMI270_BOS BMI270_BOS-M BMI270_BOS-L")
 		(sheetname "/")
@@
 			)
 		)
+		(property "LCSC Part #" "C7420338"
+			(at 0 0 180)
+			(unlocked yes)
+			(layer "F.Fab")
+			(hide yes)
+			(effects
+				(font
+					(size 1 1)
+					(thickness 0.15)
+				)
+			)
+		)
 		(property ki_fp_filters "SOT?23*")
 		(sheetname "/")
@@
 			)
 		)
-		(property "Value" "10u"
+		(property "Value" "10uF"
 			(at 0 1.68 0)
 			(layer "F.Fab")
@@
 			)
 		)
-		(property "Value" "10u"
+		(property "Value" "10uF"
 			(at 0 1.68 0)
 			(layer "F.Fab")
@@
 			)
 		)
+		(property "LCSC Part #" "C97253"
+			(at 0 0 270)
+			(unlocked yes)
+			(layer "F.Fab")
+			(hide yes)
+			(effects
+				(font
+					(size 1 1)
+					(thickness 0.15)
+				)
+			)
+		)
 		(property ki_fp_filters "SOT?23*")
 		(sheetname "/")
@@
 			)
 		)
+		(property "LCSC Part # Part #" "C7420340"
+			(at 0 0 0)
+			(unlocked yes)
+			(layer "F.Fab")
+			(hide yes)
+			(effects
+				(font
+					(size 1 1)
+					(thickness 0.15)
+				)
+			)
+		)
 		(property ki_fp_filters "SOT?23*")
 		(sheetname "/")
@@
 			)
 		)
-		(property "Value" "TBD"
+		(property "Value" "27n"
 			(at 0 1.17 0)
 			(layer "F.Fab")
@@
 			)
 		)
+		(property "Part" "LQG15HS27NJ02"
+			(at 0 0 0)
+			(unlocked yes)
+			(layer "F.Fab")
+			(hide yes)
+			(effects
+				(font
+					(size 1 1)
+					(thickness 0.15)
+				)
+			)
+		)
 		(property ki_fp_filters "Choke_* *Coil* Inductor_* L_*")
 		(sheetname "/")
@@
 			)
 		)
-		(property "Value" "10u"
+		(property "Value" "10uF"
 			(at 0 1.68 90)
 			(layer "F.Fab")
@@
 			)
 		)
-		(property "Value" "2.2u"
+		(property "Value" "2.2uF"
 			(at 0 1.16 0)
 			(layer "F.Fab")
@@
 			)
 		)
+		(property "LCSC Part #" "C6898733"
+			(at 0 0 270)
+			(unlocked yes)
+			(layer "F.Fab")
+			(hide yes)
+			(effects
+				(font
+					(size 1 1)
+					(thickness 0.15)
+				)
+			)
+		)
 		(property ki_fp_filters "ublox*MAX*")
 		(sheetname "/")
@@
 			)
 		)
+		(property "LCSC Part #" "C22418213"
+			(at 0 0 180)
+			(unlocked yes)
+			(layer "F.Fab")
+			(hide yes)
+			(effects
+				(font
+					(size 1 1)
+					(thickness 0.15)
+				)
+			)
+		)
 		(property ki_fp_filters "*BNC* *SMA* *SMB* *SMC* *Cinch* *LEMO* *UMRF* *MCX* *U.FL*")
 		(sheetname "/")
@@
 			)
 		)
-		(property "Value" "22u"
+		(property "Value" "22uF"
 			(at 0 1.68 0)
 			(layer "F.Fab")
@@
 			)
 		)
+		(property "LCSC" "C2150885"
+			(at 0 0 90)
+			(unlocked yes)
+			(layer "F.Fab")
+			(hide yes)
+			(effects
+				(font
+					(size 1 1)
+					(thickness 0.15)
+				)
+			)
+		)
 		(property ki_fp_filters "21-0164_L1022+1_MXM 21-0164B_L1022-1-M_MXM 21-0164B_L1022-1-L_MXM")
 		(sheetname "/charger/")
@@
 			)
 		)
+		(property "LCSC" "C779403"
+			(at 0 0 90)
+			(unlocked yes)
+			(layer "F.Fab")
+			(hide yes)
+			(effects
+				(font
+					(size 1 1)
+					(thickness 0.15)
+				)
+			)
+		)
 		(property ki_fp_filters "SOT?23*")
 		(sheetname "/charger/")
@@
 			)
 		)
-		(property "Value" "C_Small"
+		(property "Value" "1n"
 			(at 0 1.16 0)
 			(layer "F.Fab")
@@
 			)
 		)
+		(property "LCSC Part #" "C965555"
+			(at 0 0 185)
+			(unlocked yes)
+			(layer "B.Fab")
+			(hide yes)
+			(effects
+				(font
+					(size 1 1)
+					(thickness 0.15)
+				)
+				(justify mirror)
+			)
+		)
 		(property ki_fp_filters "LED*WS2812*-2020_PLCC4*")
 		(sheetname "/")
@@
 			)
 		)
+		(property "LCSC" "C2843970"
+			(at 0 0 180)
+			(unlocked yes)
+			(layer "B.Fab")
+			(hide yes)
+			(effects
+				(font
+					(size 1 1)
+					(thickness 0.15)
+				)
+				(justify mirror)
+			)
+		)
 		(property ki_fp_filters "USB*C*Receptacle*")
 		(sheetname "/charger/")
@@
 			(drill 0.7)
 			(property pad_prop_heatsink)
-			(layers "F&B.Cu" "*.Mask" "B.Paste")
+			(layers "*.Cu" "*.Mask" "B.Paste")
 			(remove_unused_layers no)
 			(net 8 "Net-(J3-SHIELD)")
@@
 			(drill 0.7)
 			(property pad_prop_heatsink)
-			(layers "F&B.Cu" "*.Mask" "B.Paste")
+			(layers "*.Cu" "*.Mask" "B.Paste")
 			(remove_unused_layers no)
 			(net 8 "Net-(J3-SHIELD)")
@@
 			(drill 0.7)
 			(property pad_prop_heatsink)
-			(layers "F&B.Cu" "*.Mask" "B.Paste")
+			(layers "*.Cu" "*.Mask" "B.Paste")
 			(remove_unused_layers no)
 			(net 8 "Net-(J3-SHIELD)")
@@
 			(drill 0.7)
 			(property pad_prop_heatsink)
-			(layers "F&B.Cu" "*.Mask" "B.Paste")
+			(layers "*.Cu" "*.Mask" "B.Paste")
 			(remove_unused_layers no)
 			(net 8 "Net-(J3-SHIELD)")
@@
 			)
 		)
+		(property "LCSC" "C315909"
+			(at 0 0 135)
+			(unlocked yes)
+			(layer "B.Fab")
+			(hide yes)
+			(effects
+				(font
+					(size 1 1)
+					(thickness 0.15)
+				)
+				(justify mirror)
+			)
+		)
 		(sheetname "/charger/")
 		(sheetfile "usb-fast-charger.kicad_sch")
@@
 		(polygon
 			(pts
-				(xy 143.15 73.125) (xy 149.125 73.125) (xy 149.125 73.125) (xy 152.7 73.125) (xy 152.7 70.5) (xy 143.15 70.5)
+				(xy 143.15 73.125) (xy 149.125 73.125) (xy 152.7 73.125) (xy 152.7 70.5) (xy 143.15 70.5)
 			)
 		)
