File: hardware/pebble.kicad_sch (KiCad schematic)
At the start: 130 parts, among them J1 UART, J2 GPS, J5 Conn_01x03_Pin, Q1 BSS84, Q2 BSS123, U1 TPS61023DRLR, U2 TPS563200, U3 ESP32-C6-MINI-1, U4 BMI270, U5 MAX-M8Q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

Commit message: add nix flake and initial esp32-c6 project structure with probe-rs and defmt
Parts:
- D1: LCSC Part # (none) -> C965555
- J2: LCSC Part # (none) -> C22418213
- Q1: LCSC Part # Part # (none) -> C7420340
- Q2: LCSC Part # (none) -> C7420338
- U1: LCSC Part # (none) -> C919459
- U2: LCSC Part # (none) -> C97253
- U3: LCSC Part # (none) -> C5736265
- U4: LCSC Part # (none) -> C2836813
- U5: LCSC Part # (none) -> C6898733
- U6: LCSC Part # (none) -> C17225907
Changed lines of the file:
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@@
 			)
 		)
+		(property "LCSC Part #" "C22418213"
+			(at 410.21 118.11 0)
+			(effects
+				(font
+					(size 1.27 1.27)
+				)
+				(hide yes)
+			)
+		)
 		(pin "1"
 		)
@@
 			)
 		)
+		(property "LCSC Part #" "C97253"
+			(at 140.97 38.1 0)
+			(effects
+				(font
+					(size 1.27 1.27)
+				)
+				(hide yes)
+			)
+		)
 		(pin "4"
 		)
@@
 			)
 		)
+		(property "LCSC Part #" "C6898733"
+			(at 359.41 118.11 0)
+			(effects
+				(font
+					(size 1.27 1.27)
+				)
+				(hide yes)
+			)
+		)
 		(pin "2"
 		)
@@
 			)
 		)
+		(property "LCSC Part #" "C919459"
+			(at 54.61 41.91 0)
+			(effects
+				(font
+					(size 1.27 1.27)
+				)
+				(hide yes)
+			)
+		)
 		(pin "3"
 		)
@@
 			)
 		)
+		(property "LCSC Part #" "C5736265"
+			(at 304.8 58.42 0)
+			(effects
+				(font
+					(size 1.27 1.27)
+				)
+				(hide yes)
+			)
+		)
 		(pin "37"
 		)
@@
 			)
 		)
+		(property "LCSC Part #" "C965555"
+			(at 25.4 170.18 0)
+			(effects
+				(font
+					(size 1.27 1.27)
+				)
+				(hide yes)
+			)
+		)
 		(pin "3"
 		)
@@
 			)
 		)
+		(property "LCSC Part #" "C2836813"
+			(at 355.6 224.79 0)
+			(effects
+				(font
+					(size 1.27 1.27)
+				)
+				(hide yes)
+			)
+		)
 		(pin "1"
 		)
@@
 			)
 		)
+		(property "LCSC Part #" "C7420338"
+			(at 387.35 105.41 0)
+			(effects
+				(font
+					(size 1.27 1.27)
+				)
+				(hide yes)
+			)
+		)
 		(pin "1"
 		)
@@
 			)
 		)
+		(property "LCSC Part #" "C17225907"
+			(at 359.41 168.91 0)
+			(effects
+				(font
+					(size 1.27 1.27)
+				)
+				(hide yes)
+			)
+		)
 		(pin "A2"
 		)
@@
 			(effects
 				(font
+					(size 1.27 1.27)
+				)
+				(hide yes)
+			)
+		)
+		(property "LCSC Part # Part #" "C7420340"
+			(at 383.54 90.17 90)
+			(effects
+				(font
